File: atlas-flight-controller-board/power.kicad_sch (KiCad schematic)
At the start: 0 parts

Commit message: Added Regulator, Leaving disconnected, and off pcb for now as teensy board does this automatically. Leaving on for future revs without teensy board
Parts:
- added C10: 33 uF, symbol Device:C_Small
- added C9: .47 uF, symbol Device:C_Small
- added J4: 5V Input Power, TerminalBlock:TerminalBlock_Xinya_XY308-2.54-2P_1x02_P2.54mm_Horizontal, symbol Connector:Screw_Terminal_01x02
- added U3: LM3940IMPX-3.3_NOPB, LM3940IMPX-3.3_NOPB:SOT230P700X180-4N, symbol LM3940IMPX-3.3_NOPB:LM3940IMPX-3.3_NOPB
Connections:
- new net +3V3: C10.1, U3.3 (OUT)
- new net +5V: C9.1, J4.2 (Pin_2), U3.1 (IN)
- new net GND: C10.2, C9.2, J4.1 (Pin_1), U3.2 (GND), U3.4 (GND)

Commit message: Wip commit
Changed lines of the file:
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@@
+	(wire
+		(pts
+			(xy 67.31 45.72) (xy 67.31 46.99)
+		)
+		(stroke
+			(width 0)
+			(type default)
+		)
+	)
 	(wire
 		(pts
@@
 	(symbol
 		(lib_id "power:+5V")
-		(at 67.31 46.99 0)
+		(at 67.31 45.72 0)
 		(unit 1)
 		(exclude_from_sim no)
@@
 		(fields_autoplaced yes)
 		(property "Reference" "#PWR07"
-			(at 67.31 50.8 0)
+			(at 67.31 49.53 0)
 			(effects
 				(font
@@
 		)
 		(property "Value" "+5V"
-			(at 67.31 41.91 0)
+			(at 67.31 40.64 0)
 			(effects
 				(font
@@
 		)
 		(property "Footprint" ""
-			(at 67.31 46.99 0)
+			(at 67.31 45.72 0)
 			(effects
 				(font
@@
 		)
 		(property "Datasheet" ""
-			(at 67.31 46.99 0)
+			(at 67.31 45.72 0)
 			(effects
 				(font
@@
 		)
 		(property "Description" "Power symbol creates a global label with name \"+5V\""
-			(at 67.31 46.99 0)
+			(at 67.31 45.72 0)
 			(effects
 				(font

Commit message: wip with saves
Other:
- moved on the sheet: J4
Changed lines of the file:
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@@
 	(wire
 		(pts
-			(xy 67.31 58.42) (xy 67.31 49.53)
-		)
-		(stroke
-			(width 0)
-			(type default)
-		)
-	)
-	(wire
-		(pts
-			(xy 59.69 46.99) (xy 67.31 46.99)
+			(xy 41.91 46.99) (xy 67.31 46.99)
 		)
 		(stroke
@@
 	(wire
 		(pts
-			(xy 67.31 49.53) (xy 59.69 49.53)
+			(xy 48.26 49.53) (xy 41.91 49.53)
+		)
+		(stroke
+			(width 0)
+			(type default)
+		)
+	)
+	(wire
+		(pts
+			(xy 48.26 58.42) (xy 48.26 49.53)
+		)
+		(stroke
+			(width 0)
+			(type default)
+		)
+	)
+	(wire
+		(pts
+			(xy 67.31 58.42) (xy 48.26 58.42)
 		)
 		(stroke
@@
 	(symbol
 		(lib_id "Connector:Screw_Terminal_01x02")
-		(at 54.61 49.53 180)
+		(at 36.83 49.53 180)
 		(unit 1)
 		(exclude_from_sim no)
@@
 		(fields_autoplaced yes)
 		(property "Reference" "J4"
-			(at 54.61 40.64 0)
+			(at 36.83 40.64 0)
 			(effects
 				(font
@@
 		)
 		(property "Value" "5V Input Power"
-			(at 54.61 43.18 0)
+			(at 36.83 43.18 0)
 			(effects
 				(font
@@
 		)
 		(property "Footprint" "TerminalBlock:TerminalBlock_Xinya_XY308-2.54-2P_1x02_P2.54mm_Horizontal"
-			(at 54.61 49.53 0)
+			(at 36.83 49.53 0)
 			(effects
 				(font
@@
 		)
 		(property "Datasheet" "~"
-			(at 54.61 49.53 0)
+			(at 36.83 49.53 0)
 			(effects
 				(font
@@
 		)
 		(property "Description" "Generic screw terminal, single row, 01x02, script generated (kicad-library-utils/schlib/autogen/connector/)"
-			(at 54.61 49.53 0)
+			(at 36.83 49.53 0)
 			(effects
 				(font

Commit message: removing some olds symbols, adding some new things such as nand flash chip.
Parts:
- U3: footprint LM3940IMPX-3.3_NOPB:SOT230P700X180-4N -> LM3940IMPX-3:SOT230P700X180-4N
Changed lines of the file:
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@@
 			)
 		)
-		(property "Footprint" "LM3940IMPX-3.3_NOPB:SOT230P700X180-4N"
+		(property "Footprint" "LM3940IMPX-3:SOT230P700X180-4N"
 			(at 100.33 49.53 0)
 			(effects

Commit message: Bare Schematic (No LEDS, etc added) finished. Begin PCB Layout.
Parts:
- removed C10: 33 uF, symbol Device:C_Small
- removed C9: .47 uF, symbol Device:C_Small
- removed J4: 5V Input Power, TerminalBlock:TerminalBlock_Xinya_XY308-2.54-2P_1x02_P2.54mm_Horizontal, symbol Connector:Screw_Terminal_01x02
- removed U3: LM3940IMPX-3.3_NOPB, LM3940IMPX-3:SOT230P700X180-4N, symbol LM3940IMPX-3.3_NOPB:LM3940IMPX-3.3_NOPB
