File: atlas-flight-controller-board/atlas-flight-controller-board.kicad_pcb (KiCad board)
At the start: 2 copper layers, 17 parts, among them IC1 LSM6DSV80XTR, IC2 LPS22HHTR, J1 UART8 RPI Screw Term, J2 Ultimate GPS Breakout Socket, J3 XTSD Socket, J4 5V Input Power, U1 LIS2MDL, U2 DEV-16771

Commit message: wip commit
Parts:
- moved J2 6.59 mm to (97.3, 58.4)
- moved C2 6.59 mm to (148.9, 75.5)
- moved C6 6.59 mm to (148.9, 83.0)
- moved C8 6.59 mm to (148.9, 88.0)
- moved J3 6.59 mm to (97.5, 84.8)
- moved J4 6.59 mm to (149.4, 58.2)
- moved U2 6.59 mm to (129.3, 87.6)
- moved C1 6.59 mm to (148.9, 73.0)
- moved C4 6.59 mm to (148.9, 78.0)
- moved C5 6.59 mm to (148.9, 80.5)
- moved C7 6.59 mm to (148.9, 85.5)
- moved J1 6.59 mm to (149.6, 111.8)
- moved RFD900x1 6.59 mm to (99.3, 110.5)
Changed lines of the file:
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@@
 	(footprint "Capacitor_SMD:C_0603_1608Metric_Pad1.08x0.95mm_HandSolder"
 		(layer "F.Cu")
-		(at 155.2368 77.2552)
+		(at 148.8868 75.4772)
 		(descr "Capacitor SMD 0603 (1608 Metric), square (rectangular) end terminal, IPC-7351 nominal with elongated pad for handsoldering. (Body size source: IPC-SM-782 page 76, https://www.pcb-3d.com/wordpress/wp-content/uploads/ipc-sm-782a_amendment_1_and_2.pdf), generated with kicad-footprint-generator")
 		(tags "capacitor handsolder")
@@
 	(footprint "TerminalBlock:TerminalBlock_Xinya_XY308-2.54-2P_1x02_P2.54mm_Horizontal"
 		(layer "F.Cu")
-		(at 155.956 113.538 -90)
+		(at 149.606 111.76 -90)
 		(descr "Terminal Block Xinya XY308-2.54-2P, 2 pins, pitch 2.54mm, size 5.58x6.5mm, drill diameter 1.2mm, pad diameter 2mm, http://www.xinyaelectronic.com/product/xy308-254, script-generated using https://gitlab.com/kicad/libraries/kicad-footprint-generator/-/tree/master/scripts/TerminalBlock_Xinya")
 		(tags "THT Terminal Block Xinya XY308-2.54-2P pitch 2.54mm size 5.58x6.5mm drill 1.2mm pad 2mm")
@@
 	(footprint "Capacitor_SMD:C_0603_1608Metric_Pad1.08x0.95mm_HandSolder"
 		(layer "F.Cu")
-		(at 155.2368 84.7852)
+		(at 148.8868 83.0072)
 		(descr "Capacitor SMD 0603 (1608 Metric), square (rectangular) end terminal, IPC-7351 nominal with elongated pad for handsoldering. (Body size source: IPC-SM-782 page 76, https://www.pcb-3d.com/wordpress/wp-content/uploads/ipc-sm-782a_amendment_1_and_2.pdf), generated with kicad-footprint-generator")
 		(tags "capacitor handsolder")
@@
 	(footprint "TerminalBlock:TerminalBlock_Xinya_XY308-2.54-2P_1x02_P2.54mm_Horizontal"
 		(layer "F.Cu")
-		(at 155.702 59.944 -90)
+		(at 149.352 58.166 -90)
 		(descr "Terminal Block Xinya XY308-2.54-2P, 2 pins, pitch 2.54mm, size 5.58x6.5mm, drill diameter 1.2mm, pad diameter 2mm, http://www.xinyaelectronic.com/product/xy308-254, script-generated using https://gitlab.com/kicad/libraries/kicad-footprint-generator/-/tree/master/scripts/TerminalBlock_Xinya")
 		(tags "THT Terminal Block Xinya XY308-2.54-2P pitch 2.54mm size 5.58x6.5mm drill 1.2mm pad 2mm")
@@
 	(footprint "Capacitor_SMD:C_0603_1608Metric_Pad1.08x0.95mm_HandSolder"
 		(layer "F.Cu")
-		(at 155.2368 89.8052)
+		(at 148.8868 88.0272)
 		(descr "Capacitor SMD 0603 (1608 Metric), square (rectangular) end terminal, IPC-7351 nominal with elongated pad for handsoldering. (Body size source: IPC-SM-782 page 76, https://www.pcb-3d.com/wordpress/wp-content/uploads/ipc-sm-782a_amendment_1_and_2.pdf), generated with kicad-footprint-generator")
 		(tags "capacitor handsolder")
@@
 	(footprint "Connector_PinSocket_2.54mm:PinSocket_1x07_P2.54mm_Vertical"
 		(layer "F.Cu")
-		(at 103.886 86.614)
+		(at 97.536 84.836)
 		(descr "Through hole straight socket strip, 1x07, 2.54mm pitch, single row (from Kicad 4.0.7), script generated")
 		(tags "Through hole socket strip THT 1x07 2.54mm single row")
@@
 	(footprint "Capacitor_SMD:C_0603_1608Metric_Pad1.08x0.95mm_HandSolder"
 		(layer "F.Cu")
-		(at 155.2368 87.2952)
+		(at 148.8868 85.5172)
 		(descr "Capacitor SMD 0603 (1608 Metric), square (rectangular) end terminal, IPC-7351 nominal with elongated pad for handsoldering. (Body size source: IPC-SM-782 page 76, https://www.pcb-3d.com/wordpress/wp-content/uploads/ipc-sm-782a_amendment_1_and_2.pdf), generated with kicad-footprint-generator")
 		(tags "capacitor handsolder")
@@
 	(footprint "Capacitor_SMD:C_0603_1608Metric_Pad1.08x0.95mm_HandSolder"
 		(layer "F.Cu")
-		(at 155.2368 74.7452)
+		(at 148.8868 72.9672)
 		(descr "Capacitor SMD 0603 (1608 Metric), square (rectangular) end terminal, IPC-7351 nominal with elongated pad for handsoldering. (Body size source: IPC-SM-782 page 76, https://www.pcb-3d.com/wordpress/wp-content/uploads/ipc-sm-782a_amendment_1_and_2.pdf), generated with kicad-footprint-generator")
 		(tags "capacitor handsolder")
@@
 	(footprint "TerminalBlock:TerminalBlock_Xinya_XY308-2.54-2P_1x02_P2.54mm_Horizontal"
 		(layer "F.Cu")
-		(at 105.6355 112.273 90)
+		(at 99.2855 110.495 90)
 		(descr "Terminal Block Xinya XY308-2.54-2P, 2 pins, pitch 2.54mm, size 5.58x6.5mm, drill diameter 1.2mm, pad diameter 2mm, http://www.xinyaelectronic.com/product/xy308-254, script-generated using https://gitlab.com/kicad/libraries/kicad-footprint-generator/-/tree/master/scripts/TerminalBlock_Xinya")
 		(tags "THT Terminal Block Xinya XY308-2.54-2P pitch 2.54mm size 5.58x6.5mm drill 1.2mm pad 2mm")
@@
 	(footprint "Teensy4.1:MODULE_DEV-16771"
 		(layer "F.Cu")
-		(at 135.636 89.408 -90)
+		(at 129.286 87.63 -90)
 		(property "Reference" "U2"
 			(at 4.953 -6.977 90)
@@
 	(footprint "Capacitor_SMD:C_0603_1608Metric_Pad1.08x0.95mm_HandSolder"
 		(layer "F.Cu")
-		(at 155.2368 82.2752)
+		(at 148.8868 80.4972)
 		(descr "Capacitor SMD 0603 (1608 Metric), square (rectangular) end terminal, IPC-7351 nominal with elongated pad for handsoldering. (Body size source: IPC-SM-782 page 76, https://www.pcb-3d.com/wordpress/wp-content/uploads/ipc-sm-782a_amendment_1_and_2.pdf), generated with kicad-footprint-generator")
 		(tags "capacitor handsolder")
@@
 	(footprint "Connector_PinHeader_2.54mm:PinHeader_1x09_P2.54mm_Vertical"
 		(layer "F.Cu")
-		(at 103.632 60.198)
+		(at 97.282 58.42)
 		(descr "Through hole straight pin header, 1x09, 2.54mm pitch, single row")
 		(tags "Through hole pin header THT 1x09 2.54mm single row")
@@
 	(footprint "Capacitor_SMD:C_0603_1608Metric_Pad1.08x0.95mm_HandSolder"
 		(layer "F.Cu")
-		(at 155.2368 79.7652)
+		(at 148.8868 77.9872)
 		(descr "Capacitor SMD 0603 (1608 Metric), square (rectangular) end terminal, IPC-7351 nominal with elongated pad for handsoldering. (Body size source: IPC-SM-782 page 76, https://www.pcb-3d.com/wordpress/wp-content/uploads/ipc-sm-782a_amendment_1_and_2.pdf), generated with kicad-footprint-generator")
 		(tags "capacitor handsolder")

Commit message: Wip commit
Parts:
- moved IC1 3.65 mm to (157.5, 82.2)
- moved J1 3.05 mm to (146.6, 111.8)
- moved U2 1.63 mm to (128.3, 86.4)
Changed lines of the file:
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@@
 	(footprint "LSM6DSV80X:LSM6DSV16BXTR"
 		(layer "F.Cu")
-		(at 160.2618 84.5502)
+		(at 157.48 82.18)
 		(descr "LGA-14L 2.5 x 3.0 x 0.74 mm XDM)")
 		(tags "Integrated Circuit")
@@
 	(footprint "TerminalBlock:TerminalBlock_Xinya_XY308-2.54-2P_1x02_P2.54mm_Horizontal"
 		(layer "F.Cu")
-		(at 149.606 111.76 -90)
+		(at 146.558 111.76 -90)
 		(descr "Terminal Block Xinya XY308-2.54-2P, 2 pins, pitch 2.54mm, size 5.58x6.5mm, drill diameter 1.2mm, pad diameter 2mm, http://www.xinyaelectronic.com/product/xy308-254, script-generated using https://gitlab.com/kicad/libraries/kicad-footprint-generator/-/tree/master/scripts/TerminalBlock_Xinya")
 		(tags "THT Terminal Block Xinya XY308-2.54-2P pitch 2.54mm size 5.58x6.5mm drill 1.2mm pad 2mm")
@@
 	(footprint "Teensy4.1:MODULE_DEV-16771"
 		(layer "F.Cu")
-		(at 129.286 87.63 -90)
+		(at 128.27 86.36 -90)
 		(property "Reference" "U2"
 			(at 4.953 -6.977 90)

Commit message: wip with saves
Parts:
- moved C8 9.79 mm to (148.2, 97.8)
- moved C7 7.44 mm to (148.2, 92.9)
- moved C6 5.10 mm to (148.2, 88.1)
- moved C1 4.44 mm to (148.2, 68.6)
- moved C5 2.78 mm to (148.2, 83.2)
- moved C2 2.15 mm to (148.2, 73.4)
- moved C4 0.78 mm to (148.2, 78.3)
Changed lines of the file:
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@@
 	(footprint "Capacitor_SMD:C_0603_1608Metric_Pad1.08x0.95mm_HandSolder"
 		(layer "F.Cu")
-		(at 148.8868 75.4772)
+		(at 148.1825 73.448333)
 		(descr "Capacitor SMD 0603 (1608 Metric), square (rectangular) end terminal, IPC-7351 nominal with elongated pad for handsoldering. (Body size source: IPC-SM-782 page 76, https://www.pcb-3d.com/wordpress/wp-content/uploads/ipc-sm-782a_amendment_1_and_2.pdf), generated with kicad-footprint-generator")
 		(tags "capacitor handsolder")
@@
 	(footprint "Capacitor_SMD:C_0603_1608Metric_Pad1.08x0.95mm_HandSolder"
 		(layer "F.Cu")
-		(at 148.8868 83.0072)
+		(at 148.1825 88.053333)
 		(descr "Capacitor SMD 0603 (1608 Metric), square (rectangular) end terminal, IPC-7351 nominal with elongated pad for handsoldering. (Body size source: IPC-SM-782 page 76, https://www.pcb-3d.com/wordpress/wp-content/uploads/ipc-sm-782a_amendment_1_and_2.pdf), generated with kicad-footprint-generator")
 		(tags "capacitor handsolder")
@@
 	(footprint "Capacitor_SMD:C_0603_1608Metric_Pad1.08x0.95mm_HandSolder"
 		(layer "F.Cu")
-		(at 148.8868 88.0272)
+		(at 148.1825 97.79)
 		(descr "Capacitor SMD 0603 (1608 Metric), square (rectangular) end terminal, IPC-7351 nominal with elongated pad for handsoldering. (Body size source: IPC-SM-782 page 76, https://www.pcb-3d.com/wordpress/wp-content/uploads/ipc-sm-782a_amendment_1_and_2.pdf), generated with kicad-footprint-generator")
 		(tags "capacitor handsolder")
@@
 	(footprint "Capacitor_SMD:C_0603_1608Metric_Pad1.08x0.95mm_HandSolder"
 		(layer "F.Cu")
-		(at 148.8868 85.5172)
+		(at 148.1825 92.921667)
 		(descr "Capacitor SMD 0603 (1608 Metric), square (rectangular) end terminal, IPC-7351 nominal with elongated pad for handsoldering. (Body size source: IPC-SM-782 page 76, https://www.pcb-3d.com/wordpress/wp-content/uploads/ipc-sm-782a_amendment_1_and_2.pdf), generated with kicad-footprint-generator")
 		(tags "capacitor handsolder")
@@
 	(footprint "Capacitor_SMD:C_0603_1608Metric_Pad1.08x0.95mm_HandSolder"
 		(layer "F.Cu")
-		(at 148.8868 72.9672)
+		(at 148.1825 68.58)
 		(descr "Capacitor SMD 0603 (1608 Metric), square (rectangular) end terminal, IPC-7351 nominal with elongated pad for handsoldering. (Body size source: IPC-SM-782 page 76, https://www.pcb-3d.com/wordpress/wp-content/uploads/ipc-sm-782a_amendment_1_and_2.pdf), generated with kicad-footprint-generator")
 		(tags "capacitor handsolder")
@@
 	(footprint "Capacitor_SMD:C_0603_1608Metric_Pad1.08x0.95mm_HandSolder"
 		(layer "F.Cu")
-		(at 148.8868 80.4972)
+		(at 148.1825 83.185)
 		(descr "Capacitor SMD 0603 (1608 Metric), square (rectangular) end terminal, IPC-7351 nominal with elongated pad for handsoldering. (Body size source: IPC-SM-782 page 76, https://www.pcb-3d.com/wordpress/wp-content/uploads/ipc-sm-782a_amendment_1_and_2.pdf), generated with kicad-footprint-generator")
 		(tags "capacitor handsolder")
@@
 	(footprint "Capacitor_SMD:C_0603_1608Metric_Pad1.08x0.95mm_HandSolder"
 		(layer "F.Cu")
-		(at 148.8868 77.9872)
+		(at 148.1825 78.316667)
 		(descr "Capacitor SMD 0603 (1608 Metric), square (rectangular) end terminal, IPC-7351 nominal with elongated pad for handsoldering. (Body size source: IPC-SM-782 page 76, https://www.pcb-3d.com/wordpress/wp-content/uploads/ipc-sm-782a_amendment_1_and_2.pdf), generated with kicad-footprint-generator")
 		(tags "capacitor handsolder")

Commit message: removing some olds symbols, adding some new things such as nand flash chip.
Parts:
- removed J1: UART8 RPI Screw Term, TerminalBlock:TerminalBlock_Xinya_XY308-2.54-2P_1x02_P2.54mm_Horizontal
- removed J3: XTSD Socket, Connector_PinSocket_2.54mm:PinSocket_1x07_P2.54mm_Vertical
- added U3: LM3940IMPX-3.3_NOPB, LM3940IMPX-3:SOT230P700X180-4N, F.Cu at (169.8, 59.7)
- added U4: ~, ZDSD16GLGIAG:LGA-8_8x6.2mm_P1.27mm, F.Cu at (108.0, 90.2)
- moved IC1 1.32 mm to (156.2, 82.5)
Connections:
- IC1 pad 1: GND -> MISO_1
- IC1 pad 12: +3V3 -> CS_IMU
- IC1 pad 13: I2C_SCL -> SCK_1
- IC1 pad 14: I2C_SDA -> MOSI_1
- IC2 pad 2: I2C_SCL -> SCK_1
- IC2 pad 4: I2C_SDA -> MOSI_1
- IC2 pad 5: GND -> MISO_1
- IC2 pad 6: +3V3 -> CS_BARO
- U1 pad 1: I2C_SCL -> SCK_1
- U1 pad 3: +3V3 -> CS_MAG
- U1 pad 4: I2C_SDA -> MOSI_1
- U1 pad 7: MAG_INT -> MISO_1
- U2 pad 18: I2C_SDA -> unconnected-(U2-A4-Pad18)
- U2 pad 19: I2C_SCL -> unconnected-(U2-A5-Pad19)
- U2 pad 20: MAG_INT -> unconnected-(U2-A6-Pad20)
- U2 pad 34: /mcu-page/UART_RPI_TX_MCU_RX -> unconnected-(U2-RX8-Pad34)
- U2 pad 35: /mcu-page/UART_MCU_TX_RPI_RX -> unconnected-(U2-TX8-Pad35)
Other:
- copper layers 2 -> 4

Commit message: Bare Schematic (No LEDS, etc added) finished. Begin PCB Layout.
Parts:
- removed U3: LM3940IMPX-3.3_NOPB, LM3940IMPX-3:SOT230P700X180-4N
- moved C3 33.7 mm to (156.5, 114.3)
- moved U1 30.8 mm to (150.1, 107.4), turned to 180 degrees
- moved IC2 30.5 mm to (150.1, 99.6), turned to 180 degrees
- moved C1 25.7 mm to (147.9, 94.2), turned to 180 degrees
- moved C5 23.9 mm to (157.1, 105.4)
- moved C4 22.9 mm to (152.1, 100.9), turned to 90 degrees
- moved C6 21.5 mm to (160.9, 105.4)
- moved C2 19.8 mm to (151.7, 93.0), turned to -90 degrees
- moved C7 18.9 mm to (159.6, 108.0)
- moved RFD900x1 16.4 mm to (108.0, 96.5), turned to -90 degrees
- moved IC1 11.7 mm to (148.0, 91.0)
- moved C8 4.60 mm to (149.6, 102.2), turned to 180 degrees
- moved U4 2.54 mm to (108.0, 87.6)
- moved J4 1.70 mm to (148.6, 59.7), turned to 90 degrees
Connections:
- net SD_CS renamed CS_SD
- U2 pad 21: BARO_INT -> unconnected-(U2-A7-Pad21)
- U2 pad 22: IMU_INT1 -> unconnected-(U2-A8-Pad22)
- U2 pad 23: IMU_INT2 -> unconnected-(U2-A9-Pad23)
- U2 pad 24: unconnected-(U2-A10-Pad24) -> UART_MCU_TX_RFD900_RX
- U2 pad 25: unconnected-(U2-A11-Pad25) -> UART_RFD900_TX_MCU_RX
- U2 pad 26: unconnected-(U2-A12-Pad26) -> MOSI_1
- U2 pad 27: unconnected-(U2-A13-Pad27) -> SCK_1
- U2 pad 28: UART_RFD900_TX_MCU_RX -> unconnected-(U2-RX7-Pad28)
- U2 pad 29: UART_MCU_TX_RFD900_RX -> unconnected-(U2-TX7-Pad29)
- U2 pad 3.3V_1: 3.3V -> +3V3
- U2 pad 3.3V_2: 3.3V -> +3V3
- U2 pad 3.3V_3: 3.3V -> +3V3
- U2 pad 33: unconnected-(U2-MCLK2-Pad33) -> BARO_INT
- U2 pad 34: unconnected-(U2-RX8-Pad34) -> IMU_INT2
- U2 pad 35: unconnected-(U2-TX8-Pad35) -> IMU_INT1
- U2 pad 36: unconnected-(U2-CS2-Pad36) -> CS_IMU
- U2 pad 37: unconnected-(U2-CS3-Pad37) -> CS_BARO
- U2 pad 38: unconnected-(U2-A14-Pad38) -> CS_MAG
- U2 pad 39: unconnected-(U2-A15-Pad39) -> MISO_1
- U2 pad USB_GND1: USB_GND -> GND
- U2 pad USB_GND2: USB_GND -> GND
- U2 pad VIN: unconnected-(U2-PadVIN) -> +5V
Other:
- board text added: "Caps: IMU BARO MAG"

Commit message: Re-arranging components, trying out different SPI routings
Parts:
- moved J2 30.3 mm to (95.2, 88.6), turned to 90 degrees
- moved C6 17.1 mm to (143.8, 106.2)
- moved C7 16.2 mm to (143.8, 111.3), turned to 180 degrees
- moved RFD900x1 14.7 mm to (97.0, 106.4)
- moved C5 11.3 mm to (146.3, 108.7), turned to 90 degrees
- moved U4 9.63 mm to (108.8, 97.2)
- moved C2 8.41 mm to (146.8, 99.8)
- moved IC1 8.10 mm to (143.6, 97.8)
- moved C3 7.89 mm to (151.1, 108.5), turned to -90 degrees
- moved C1 7.56 mm to (143.8, 100.6)
- moved U1 6.47 mm to (143.8, 108.7), turned to 0 degrees
- moved C4 1.73 mm to (153.7, 101.5), turned to -90 degrees
- moved C8 1.61 mm to (151.2, 102.2)
- moved IC2 1.31 mm to (151.4, 99.6)
Connections:
- C3 pad 1: (no net) -> +3V3
- C3 pad 2: (no net) -> GND
Routing:
- net SCK: track 0.00 -> 30.9 mm
- net CS_SD: track 0.00 -> 23.1 mm, vias 0 -> 1
- net MISO: track 0.00 -> 13.9 mm
- net GND: track 0.00 -> 12.7 mm
- net +5V: track 0.00 -> 12.7 mm
- net MOSI: track 0.00 -> 12.3 mm
Other:
- board text added: "GPS"
- board text removed: "Caps: IMU BARO MAG"

Commit message: Should have SPI routed in demo, need to implement.
Parts:
- added C1: 100 nF, Capacitor_SMD:C_0603_1608Metric_Pad1.08x0.95mm_HandSolder, F.Cu at (57.9, 92.8)
- added C1: 100 nF, Capacitor_SMD:C_0603_1608Metric_Pad1.08x0.95mm_HandSolder, F.Cu at (99.7, 97.3)
- added C2: 100 nF, Capacitor_SMD:C_0603_1608Metric_Pad1.08x0.95mm_HandSolder, F.Cu at (102.8, 96.5)
- added C2: 100 nF, Capacitor_SMD:C_0603_1608Metric_Pad1.08x0.95mm_HandSolder, F.Cu at (58.7, 95.9)
- added C3: 10 uF, APA0606100M050R:CAP_APA_0606_AVX, F.Cu at (92.4, 115.3)
- added C3: 10 uF, APA0606100M050R:CAP_APA_0606_AVX, F.Cu at (54.1, 107.2)
- added C4: 100 nF, Capacitor_SMD:C_0603_1608Metric_Pad1.08x0.95mm_HandSolder, F.Cu at (98.3, 102.4)
- added C4: 100 nF, Capacitor_SMD:C_0603_1608Metric_Pad1.08x0.95mm_HandSolder, F.Cu at (59.7, 101.6)
- added C5: 100 nF, Capacitor_SMD:C_0603_1608Metric_Pad1.08x0.95mm_HandSolder, F.Cu at (92.2, 110.5)
- added C5: 100 nF, Capacitor_SMD:C_0603_1608Metric_Pad1.08x0.95mm_HandSolder, F.Cu at (58.9, 106.9)
- added C6: 100 nF, Capacitor_SMD:C_0603_1608Metric_Pad1.08x0.95mm_HandSolder, F.Cu at (94.7, 108.0)
- added C6: 100 nF, Capacitor_SMD:C_0603_1608Metric_Pad1.08x0.95mm_HandSolder, F.Cu at (61.5, 109.5)
- added C7: 220 nF, Capacitor_SMD:C_0603_1608Metric_Pad1.08x0.95mm_HandSolder, F.Cu at (61.5, 104.4)
- added C7: 220 nF, Capacitor_SMD:C_0603_1608Metric_Pad1.08x0.95mm_HandSolder, F.Cu at (89.7, 107.9)
- added C8: 100 nF, Capacitor_SMD:C_0603_1608Metric_Pad1.08x0.95mm_HandSolder, F.Cu at (95.8, 103.2)
- added C8: 100 nF, Capacitor_SMD:C_0603_1608Metric_Pad1.08x0.95mm_HandSolder, F.Cu at (58.9, 99.1)
- added IC1: LSM6DSV80XTR, LSM6DSV80X:LSM6DSV16BXTR, F.Cu at (60.8, 92.7)
- added IC1: LSM6DSV80XTR, LSM6DSV80X:LSM6DSV16BXTR, F.Cu at (99.6, 94.5)
- added IC2: LPS22HHTR, LPS22HHTR:LPS22HHTR, F.Cu at (96.0, 100.6)
- added IC2: LPS22HHTR, LPS22HHTR:LPS22HHTR, F.Cu at (61.5, 99.3)
- added U1: LIS2MDL, LIS2MDL:PQFN50P200X200X70-12N, F.Cu at (61.5, 106.9)
- added U1: LIS2MDL, LIS2MDL:PQFN50P200X200X70-12N, F.Cu at (92.2, 108.0)
- moved RFD900x1 11.9 mm to (109.0, 106.2)
Routing:
- net MISO_1: track 0.00 -> 49.0 mm, vias 0 -> 6
- net SCK_1: track 0.05 -> 49.0 mm, vias 0 -> 6
- net MOSI_1: track 0.00 -> 45.8 mm, vias 0 -> 6
- net GND: track 12.7 -> 21.6 mm, vias 0 -> 3
- net +3V3: track 0.00 -> 5.20 mm, vias 0 -> 1
- net Net-(U1-C1): track 0.00 -> 3.34 mm, vias 0 -> 1
Other:
- board text added: "NEED Resistors on MISO MOSI to figure out ringing"

Commit message: wip commit
Parts:
- moved C5 39.6 mm to (125.2, 142.2)
- moved C2 39.6 mm to (125.7, 133.3)
- moved C3 39.6 mm to (130.0, 142.0)
- moved C1 39.6 mm to (122.7, 134.1)
- moved C4 39.6 mm to (132.6, 135.1)
- moved U1 39.6 mm to (122.7, 142.2)
- moved C7 39.6 mm to (122.7, 144.8)
- moved C8 39.6 mm to (130.1, 135.7)
- moved IC2 39.6 mm to (130.3, 133.1)
- moved C6 39.6 mm to (122.7, 139.7)
- moved IC1 39.6 mm to (122.5, 131.3)
- moved C1 39.1 mm to (97.0, 94.9)
- moved C2 39.1 mm to (97.8, 97.9)
- moved IC1 39.1 mm to (99.8, 94.7)
- moved C7 38.6 mm to (100.0, 106.7)
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Routing:
- net GND: track 21.6 -> 38.5 mm, vias 3 -> 7
- net +3V3: track 5.20 -> 19.6 mm, vias 1 -> 4
- net Net-(U1-C1): track 3.34 -> 5.22 mm
- net CS_MAG: track 0.00 -> 1.48 mm, vias 0 -> 1
- net MISO_1: track 49.0 -> 47.9 mm
- net SCK_1: track 49.0 -> 48.2 mm
- net MOSI_1: track 45.8 -> 45.0 mm
